Commit message: joint_states_and_ros2_control_issue

File: src/robot_description/urdf/manipulaor_ros2_control.xacro (robot description, xacro)
@@ -3,7 +3,7 @@
     <xacro:property name="PI" value="3.14159"/>
     <ros2_control type="system" name="RobotSystem">
-            <hardware>
-                <plugin>gz_ros2_control/GazeboSimSystem</plugin> <!-- Ignition Gazebo ROS2 humble control plugin -->
-            </hardware>
+        <hardware>
+            <plugin>gz_ros2_control/GazeboSimSystem</plugin> <!-- Ignition Gazebo ROS2 humble control plugin -->
+        </hardware>
         <!-- Joints Configuration -->
         <joint name="basement_to_base_plate">

File: src/robot_description/urdf/manipulator.urdf.xacro (robot description, xacro)
@@ -3,9 +3,9 @@
 <!-- Name of the robot is "manipulator" -->
 <robot name="manipulator" xmlns:xacro="http://ros.org/wiki/xacro">
-    <xacro:arg name="is_ignition" default="true"/>
+    <!-- <xacro:arg name="is_ignition" default="true"/>  -->
     <!--this arg is used to load proper ros2 control plugin-->
     <xacro:include filename="$(find robot_description)/urdf/manipulator_gazebo.xacro"/>
     <xacro:include filename="$(find robot_description)/urdf/manipulator_ros2_control.xacro"/>
-     <xacro:include filename="$(find robot_description)/urdf/camera.xacro"/>
+    <xacro:include filename="$(find robot_description)/urdf/camera.xacro"/>
     <!-- Creating the variables -->
     <xacro:property name="PI" value="3.14159"/>
@@ -24,4 +24,5 @@
         <xacro:default_inertia mass="1.0"/>
         <visual>
+            <!-- Displacement and orientation  of the geometric center of the link with respect to previous link-->
             <origin xyz="-0.5 -0.5 0.0" rpy="0.0 0.0 0.0"/>
             <geometry>

File: src/robot_description/urdf/manipulator_gazebo.xacro (robot description, xacro)
@@ -3,16 +3,42 @@
     <gazebo>
         <!-- Load proper ros2 control plugin based on simulator -->
-        <xacro:if value="$(arg is_ignition)">
-            <plugin filename="ign_ros2_control-system" name="ign_ros2_control::IgnitionRos2ControlPlugin">
-                <parameters>
-                </parameters>
-            </plugin>
-        </xacro:if>
-        <xacro:unless value="$(arg is_ignition)">
-            <plugin filename="gz_ros2_control-system" name="gz_ros2_control::GazeboSimROS2ControlPlugin">
-                <parameters>
-                </parameters>
-            </plugin>
-        </xacro:unless>
+        <plugin filename="gz_ros2_control-system" name="gz_ros2_control::GazeboSimRos2ControlPlugin">
+            <parameters>$(find manipulator_controller)/config/manipulator_controller.yaml</parameters>
+        </plugin>
+    </gazebo>
+    <gazebo reference="base_link">
+        <mu1>0.2</mu1>
+        <mu2>0.2</mu2>
+        <material>Gazebo/Blue</material>
+    </gazebo>
+    <gazebo reference="base_plate">
+        <mu1>0.2</mu1>
+        <mu2>0.2</mu2>
+        <material>Gazebo/Blue</material>
+    </gazebo>
+    <gazebo reference="forward_drive_arm">
+        <mu1>0.2</mu1>
+        <mu2>0.2</mu2>
+        <material>Gazebo/Blue</material>
+    </gazebo>
+    <gazebo reference="horizontal_arm">
+        <mu1>0.2</mu1>
+        <mu2>0.2</mu2>
+        <material>Gazebo/Blue</material>
+    </gazebo>
+    <gazebo reference="claw_support">
+        <mu1>0.2</mu1>
+        <mu2>0.2</mu2>
+        <material>Gazebo/Blue</material>
+    </gazebo>
+    <gazebo reference="gripper_finger_left">
+        <mu1>0.2</mu1>
+        <mu2>0.2</mu2>
+        <material>Gazebo/Blue</material>
+    </gazebo>
+    <gazebo reference="gripper_finger_right">
+        <mu1>0.2</mu1>
+        <mu2>0.2</mu2>
+        <material>Gazebo/Blue</material>
     </gazebo>
 </robot>

Commit message: Update robot_description, ros2_control and launch files

File: src/robot_description/urdf/manipulaor_ros2_control.xacro (robot description, xacro)
@@ -1,9 +1,19 @@
 <?xml version="1.0"?>
 <robot name="manipulator" xmlns:xacro="http://ros.org/wiki/xacro">
-    <xacro:property name="PI" value="3.14159"/>
     <ros2_control type="system" name="RobotSystem">
-        <hardware>
-            <plugin>gz_ros2_control/GazeboSimSystem</plugin> <!-- Ignition Gazebo ROS2 humble control plugin -->
-        </hardware>
+        <xacro:property name="PI" value="3.14159"/>
+        <!-- ros2_control Gazebo -->
+        <!-- ROS 2 Humble -->
+        <xacro:if value="$(arg is_ignition)">
+            <hardware>
+                <plugin>ign_ros2_control/IgnitionSystem</plugin>
+            </hardware>
+        </xacro:if>
+        <!-- ROS 2 Iron or above -->
+        <xacro:unless value="$(arg is_ignition)">
+            <hardware>
+                <plugin>gz_ros2_control/GazeboSimSystem</plugin>
+            </hardware>
+        </xacro:unless>
         <!-- Joints Configuration -->
         <joint name="basement_to_base_plate">

File: src/robot_description/urdf/manipulator.urdf.xacro (robot description, xacro)
@@ -3,9 +3,8 @@
 <!-- Name of the robot is "manipulator" -->
 <robot name="manipulator" xmlns:xacro="http://ros.org/wiki/xacro">
-    <!-- <xacro:arg name="is_ignition" default="true"/>  -->
-    <!--this arg is used to load proper ros2 control plugin-->
+    <xacro:arg name="is_ignition" default="false"/>  <!--if using Gazebo Harmonic (default="false") and Gazebo Ignition (default="true") -->
+    <!-- Including other xacro files -->
     <xacro:include filename="$(find robot_description)/urdf/manipulator_gazebo.xacro"/>
     <xacro:include filename="$(find robot_description)/urdf/manipulator_ros2_control.xacro"/>
-    <xacro:include filename="$(find robot_description)/urdf/camera.xacro"/>
     <!-- Creating the variables -->
     <xacro:property name="PI" value="3.14159"/>
@@ -153,5 +152,5 @@
         </collision>
     </link>
-     <!-- CAMERA LINK
+     <!-- CAMERA LINK     -->
     <link name="rgb_camera">
         <xacro:default_inertia mass="0.01"/>
@@ -172,5 +171,4 @@
         </collision>
     </link>
-    -->
  <!-- Defining the joints between the links -->
     <!-- World to basement joint -->
@@ -228,5 +226,5 @@
         <limit lower="-${PI/2}" upper="0.0" effort="${effort}" velocity="${velocity}"/>
     </joint>
-    <!-- base_link to rgb_camera joint
+    <!-- base_link to rgb_camera joint -->
     <joint name="rgb_camera_joint" type="fixed">
         <parent link="base_link"/>
@@ -234,4 +232,3 @@
         <origin xyz="0.0 0.45 0.2" rpy="0 -0.5 1.57"/>
     </joint>
-    -->
 </robot>

File: src/robot_description/urdf/manipulator_gazebo.xacro (robot description, xacro)
@@ -1,9 +1,18 @@
 <?xml version="1.0"?>
 <robot name="manipulator" xmlns:xacro="http://ros.org/wiki/xacro">
+  <!-- ROS 2 Control -->
     <gazebo>
-        <!-- Load proper ros2 control plugin based on simulator -->
-        <plugin filename="gz_ros2_control-system" name="gz_ros2_control::GazeboSimRos2ControlPlugin">
-            <parameters>$(find manipulator_controller)/config/manipulator_controller.yaml</parameters>
-        </plugin>
+        <!-- ROS 2 Humble -->
+        <xacro:if value="$(arg is_ignition)">
+            <plugin filename="ign_ros2_control-system" name="ign_ros2_control::IgnitionROS2ControlPlugin">
+                <parameters>$(find manipulator_controller)/config/manipulator_controller.yaml</parameters>
+            </plugin>
+        </xacro:if>
+        <!-- ROS 2 Iron or above -->
+        <xacro:unless value="$(arg is_ignition)">
+            <plugin filename="gz_ros2_control-system" name="gz_ros2_control::GazeboSimROS2ControlPlugin">
+                <parameters>$(find manipulator_controller)/config/manipulator_controller.yaml</parameters>
+            </plugin>
+        </xacro:unless>
     </gazebo>
     <gazebo reference="base_link">
