Commit message: Physics properties in urdf for GAZEBO

File: src/robot_description/urdf/manipulator.urdf.xacro (robot description, xacro)
@@ -7,7 +7,15 @@
     <xacro:property name="effort" value="30.0"/>
     <xacro:property name="velocity" value="10.0"/>
+    <xacro:macro name="default_inertia" params="mass">      <!--only change the mass -->
+        <inertial>
+            <mass value="${mass}"/>
+            <inertia ixx="0.1" ixy="0.0" ixz="0.0" iyy="0.1" iyz="0.0" izz="0.1"/>
+        </inertial>
+    </xacro:macro>
     <!-- Define the robot's links and joints -->
      <link name="world"/>
     <link name="base_link">
+        <!-- Using macro file instead of whole inertial tag making it reusable -->
+        <xacro:default_inertia mass="1.0"/>
         <visual>
             <origin xyz="-0.5 -0.5 0.0" rpy="0.0 0.0 0.0"/>
@@ -19,7 +27,14 @@
             </material>
         </visual>
+        <collision>
+            <origin xyz="-0.5 -0.5 0.0" rpy="0.0 0.0 0.0"/>
+            <geometry>
+                <mesh filename="package://robot_description/meshes/basement.STL" scale="0.01 0.01 0.01"/>
+            </geometry>
+        </collision>
     </link>
     <!--2nd part-->
     <link name="base_plate">
+        <xacro:default_inertia mass="0.1"/>
         <visual>
             <origin xyz="-0.36 -0.40 -0.56" rpy="0 0 0"/>
@@ -31,7 +46,14 @@
             </material>
         </visual>
+        <collision>
+            <origin xyz="-0.36 -0.40 -0.56" rpy="0 0 0"/>
+            <geometry>
+               <mesh filename="package://robot_description/meshes/base_plate.STL" scale="0.01 0.01 0.01"/>
+            </geometry>
+        </collision>
     </link>
     <!--3rd part-->
     <link name="forward_drive_arm">
+        <xacro:default_inertia mass="0.1"/>
         <visual>
             <origin xyz="0.19 0.06 -0.08" rpy="0 -${PI/2} ${PI/2}"/>
@@ -43,7 +65,14 @@
             </material>
         </visual>
+        <collision>
+            <origin xyz="0.19 0.06 -0.08" rpy="0 -${PI/2} ${PI/2}"/>
+            <geometry>
+                <mesh filename="package://robot_description/meshes/forward_drive_arm.STL" scale="0.01 0.01 0.01"/>
+            </geometry>
+        </collision>
     </link>
     <!--4th part -->
     <link name="horizontal_arm">
+        <xacro:default_inertia mass="0.1"/>
         <visual>
             <origin xyz="-0.03 -0.4 -0.06" rpy="${PI/2} 0 ${PI/2}"/>
@@ -55,7 +84,14 @@
             </material>
         </visual>
+        <collision>
+            <origin xyz="-0.03 -0.4 -0.06" rpy="${PI/2} 0 ${PI/2}"/>
+            <geometry>
+                <mesh filename="package://robot_description/meshes/horizontal_arm.STL" scale="0.01 0.01 0.01"/>
+            </geometry>
+        </collision>
     </link>
     <!-- 5th part -->
     <link name="claw_support">
+        <xacro:default_inertia mass="0.05"/>
         <visual>
             <origin xyz="0.0 -0.05 -0.15" rpy="0 0 ${PI/2}"/>
@@ -67,7 +103,14 @@
             </material>
         </visual>
+        <collision>
+            <origin xyz="0.0 -0.05 -0.15" rpy="0 0 ${PI/2}"/>
+            <geometry>
+                <mesh filename="package://robot_description/meshes/claw_support.STL" scale="0.01 0.01 0.01"/>
+            </geometry>
+        </collision>
     </link>
     <!-- gripper fingers -->
     <link name="gripper_finger_left">
+        <xacro:default_inertia mass="0.01"/>
         <visual>
             <origin xyz="-0.04 0.5 -0.1" rpy="0 0 -${PI/2}"/>
@@ -79,6 +122,13 @@
             </material>
         </visual>
+        <collision>
+            <origin xyz="-0.04 0.5 -0.1" rpy="0 0 -${PI/2}"/>
+            <geometry>
+                <mesh filename="package://robot_description/meshes/left_finger.STL" scale="0.01 0.01 0.01"/>
+            </geometry>
+        </collision>
     </link>
     <link name="gripper_finger_right">
+        <xacro:default_inertia mass="0.01"/>
         <visual>
             <origin xyz="-0.1 0.5 -0.1" rpy="0 0 -${PI/2}"/>
@@ -90,6 +140,13 @@
             </material>
         </visual>
+        <collision>
+            <origin xyz="-0.1 0.5 -0.1" rpy="0 0 -${PI/2}"/>
+            <geometry>
+                <mesh filename="package://robot_description/meshes/right_finger.STL" scale="0.01 0.01 0.01"/>
+            </geometry>
+        </collision>
     </link>
     <link name="rgb_camera">
+        <xacro:default_inertia mass="0.01"/>
         <visual>
             <origin xyz="-0.09 0.13 0.13" rpy="-${PI*0.4888888889} 0 -${PI*0.5}"/>
@@ -101,4 +158,10 @@
             </material>
         </visual>
+        <collision>
+            <origin xyz="-0.09 0.13 0.13" rpy="-${PI*0.4888888889} 0 -${PI*0.5}"/>
+            <geometry>
+                <mesh filename="package://robot_description/meshes/pi_camera.STL" scale="0.01 0.01 0.01"/>
+            </geometry>
+        </collision>
     </link>
  <!-- Defining the joints between the links -->

Commit message: new world file and gripper finger allignment solved

File: src/robot_description/urdf/manipulator.urdf.xacro (robot description, xacro)
@@ -221,5 +221,5 @@
         <parent link="claw_support"/>
         <child link="gripper_finger_right"/>
-        <origin xyz="0.04 0.13 -0.01" rpy="0 0 0"/>
+        <origin xyz="-0.048 0.13 -0.1" rpy="0 0 0"/>
         <axis xyz="0 0 1"/> <!-- Rotation around Z-axis -->
         <mimic joint="claw_support_to_gripper_finger_left" multiplier="-1.0"/>

Commit message: fixed small bugs

File: src/robot_description/urdf/manipulator.urdf.xacro (robot description, xacro)
@@ -225,5 +225,5 @@
         <origin xyz="0.04 0.13 -0.01" rpy="0 0 0"/>
         <axis xyz="0 0 1"/> <!-- Rotation around Z-axis -->
-        <mimic joint="claw_support_to_gripper_finger_left" multiplier="-1.0"/>
+        <mimic joint="claw_support_to_gripper_finger_left" multiplier="-1"/>
         <limit lower="-${PI/2}" upper="0.0" effort="${effort}" velocity="${velocity}"/>
     </joint>

File: src/robot_description/urdf/manipulator_gazebo.xacro (robot description, xacro)
@@ -3,5 +3,5 @@
     <gazebo>
         <!-- Load proper ros2 control plugin based on simulator -->
-        <plugin filename="gz_ros2_control-system" name="gz_ros2_control::GazeboSimRos2ControlPlugin">
+        <plugin filename="gz_ros2_control-system" name="gz_ros2_control::GazeboSimROS2ControlPlugin">
             <parameters>$(find manipulator_controller)/config/manipulator_controller.yaml</parameters>
         </plugin>

File: src/robot_description/urdf/manipulator_ros2_control.xacro (robot description, xacro)
@@ -2,5 +2,5 @@
 <robot name="manipulator" xmlns:xacro="http://ros.org/wiki/xacro">
     <xacro:property name="PI" value="3.14159"/>
-    <ros2_control type="system" name="RobotSystem">
+    <ros2_control type="system" name="manipulator_controller">
         <hardware>
             <plugin>gz_ros2_control/GazeboSimSystem</plugin> <!-- Ignition Gazebo ROS2 humble control plugin -->
@@ -9,6 +9,6 @@
         <joint name="basement_to_base_plate">
             <command_interface name="position">  <!-- command interface for position control -->
-                <param name="min"> -${PI/2} </param>
-                <param name="max"> ${PI/2} </param>
+                <param name="min">-${PI/2}</param>
+                <param name="max">${PI/2}</param>
             </command_interface>
             <state_interface name="position"/>   <!-- state interface to read the position -->
@@ -16,6 +16,6 @@
         <joint name="base_plate_to_forward_drive_arm">
             <command_interface name="position">  <!-- command interface for position control -->
-                <param name="min"> -${PI/2} </param>
-                <param name="max"> ${PI/2} </param>
+                <param name="min">-${PI/2}</param>
+                <param name="max">${PI/2}</param>
             </command_interface>
             <state_interface name="position"/>   <!-- state interface to read the position -->
@@ -23,6 +23,6 @@
         <joint name="forward_drive_arm_to_horizontal_arm">
             <command_interface name="position">  <!-- command interface for position control -->
-                <param name="min"> -${PI/2} </param>
-                <param name="max"> ${PI/2} </param>
+                <param name="min">-${PI/2}</param>
+                <param name="max">${PI/2}</param>
             </command_interface>
             <state_interface name="position"/>   <!-- state interface to read the position -->
@@ -31,6 +31,6 @@
         <joint name="claw_support_to_gripper_finger_left">
             <command_interface name="position">  <!-- command interface for position control -->
-                <param name="min"> -${PI/2} </param>
-                <param name="max"> 0.0 </param>
+                <param name="min">-${PI/2}</param>
+                <param name="max">0.0</param>
             </command_interface>
             <state_interface name="position"/>   <!-- state interface to read the position -->
